File: ThumbsUpUnsplit.kicad_pcb (KiCad board)
At the start: 2 copper layers, 256.9 x 123.2 mm, 120 parts, among them J1 Conn_01x18_Male, J2 Conn_01x18_Female, J3 Conn_01x04_Female, J4 Conn_01x04_Male, J5 Conn_01x04_Female, J6 Conn_01x04_Male, J7 Conn_01x18_Female, J8 Conn_01x18_Male, SW1 SW_Push, U1 ATmega32U4-AU, Y1 16MHz

Commit message: Roughed in the connectors
Parts:
- removed the J4 at (49.1, -212.1)
- removed the J4 at (20.7, -233.2)
- removed the J6 at (112.9, -211.9)
- removed the J6 at (81.0, -255.8)
- removed the J6 at (130.5, -211.7)
- removed the J6 at (31.5, -211.6)
- removed the J6 at (141.3, -233.2)
- added J10: Raiser_Male, Connector_PinHeader_2.54mm:PinHeader_1x04_P2.54mm_Vertical, F.Cu at (130.5, -211.7)
- added J11: Raiser_Female, Connector_PinSocket_2.54mm:PinSocket_1x04_P2.54mm_Vertical, B.Cu at (32.0, -95.0)
- added J12: Raiser_Male, Connector_PinHeader_2.54mm:PinHeader_1x04_P2.54mm_Vertical, F.Cu at (31.5, -211.6)
- added J13: Raiser_Female, Connector_PinSocket_2.54mm:PinSocket_1x04_P2.54mm_Vertical, B.Cu at (81.5, -20.3)
- added J14: Raiser_Male, Connector_PinHeader_2.54mm:PinHeader_1x04_P2.54mm_Vertical, F.Cu at (81.5, -139.2)
- added J15: Raiser_Female, Connector_PinSocket_2.54mm:PinSocket_1x04_P2.54mm_Vertical, B.Cu at (113.4, 23.6)
- added J16: Raiser_Male, Connector_PinHeader_2.54mm:PinHeader_1x04_P2.54mm_Vertical, F.Cu at (113.4, -95.3)
- added J17: Raiser_Female, Connector_PinSocket_2.54mm:PinSocket_1x04_P2.54mm_Vertical, B.Cu at (49.6, 23.3)
- added J18: Raiser_Male, Connector_PinHeader_2.54mm:PinHeader_1x04_P2.54mm_Vertical, F.Cu at (49.6, -95.5)
- added J4: Conn_01x04_Male, Connector_PinHeader_2.54mm:PinHeader_1x04_P2.54mm_Vertical, B.Cu at (21.2, 2.26)
- added J6: Conn_01x04_Male, Connector_PinHeader_2.54mm:PinHeader_1x04_P2.54mm_Vertical, B.Cu at (141.8, 2.26)
- added J9: Raiser_Female, Connector_PinSocket_2.54mm:PinSocket_1x04_P2.54mm_Vertical, B.Cu at (131.0, -95.1)
- J2, J7: moved to B.Cu
- moved MX22 235.5 mm to (41.5, 20.7)
- moved MX26 235.5 mm to (121.6, 20.7)
- moved MX18 235.5 mm to (26.3, 9.22)
- moved MX30 235.5 mm to (136.7, 9.22)
- moved J2 116.6 mm to (42.6, -172.3), turned to 156 degrees
- moved J7 116.6 mm to (120.4, -172.3), turned to 202 degrees
- moved MX15 116.6 mm to (48.3, -165.0)
- moved MX16 116.6 mm to (41.2, -147.4)
- moved MX17 116.6 mm to (34.1, -129.7)
- moved MX27 116.6 mm to (114.7, -165.0)
- moved MX28 116.6 mm to (121.8, -147.4)
- moved MX29 116.6 mm to (129.0, -129.7)
- moved MX21 116.6 mm to (52.8, -125.4)
- moved MX25 116.6 mm to (110.2, -125.4)
- moved J3 116.6 mm to (21.2, -116.6)
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Other:
- board size 256.9 x 123.2 mm -> 256.9 x 358.6 mm

Commit message: Bottom plate routed
Parts:
- J3, J5: moved to B.Cu
- J4, J6: moved to F.Cu
- moved SW1 394.5 mm to (98.0, -88.0)
- moved USB1 349.1 mm to (181.0, -153.0)
- moved Y1 312.3 mm to (77.0, -93.0)
- moved U1 267.8 mm to (81.0, -107.0)
- moved C1 204.1 mm to (-20.3, -152.0)
- moved C10 204.1 mm to (-15.9, -152.0)
- moved C2 204.1 mm to (-2.64, -152.0)
- moved C3 204.1 mm to (1.77, -152.0)
- moved C4 204.1 mm to (6.18, -152.0)
- moved C5 204.1 mm to (10.6, -155.3)
- moved C6 204.1 mm to (15.0, -155.3)
- moved C7 204.1 mm to (-24.7, -152.0)
- moved C8 204.1 mm to (-7.05, -152.0)
- moved C9 204.1 mm to (-11.5, -152.0)
- moved D11 204.1 mm to (-12.8, -155.1)
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Connections:
- J3 pad 1: COL6 -> Net-(J3-Pad1)
- J3 pad 2: Net-(D19-Pad2) -> Net-(J3-Pad2)
- J3 pad 3: Net-(D18-Pad2) -> Net-(J3-Pad3)
- J3 pad 4: COL7 -> Net-(J3-Pad4)
- J4 pad 1: Net-(J4-Pad1) -> (no net)
- J4 pad 2: Net-(J4-Pad2) -> (no net)
- J4 pad 3: Net-(J4-Pad3) -> (no net)
- J4 pad 4: Net-(J4-Pad4) -> (no net)
- J5 pad 1: COL4 -> Net-(J5-Pad1)
- J5 pad 2: Net-(D30-Pad2) -> Net-(J5-Pad2)
- J5 pad 3: Net-(D29-Pad2) -> Net-(J5-Pad3)
- J5 pad 4: COL5 -> Net-(J5-Pad4)
- J6 pad 1: Net-(J6-Pad1) -> (no net)
- J6 pad 2: Net-(J6-Pad2) -> (no net)
- J6 pad 3: Net-(J6-Pad3) -> (no net)
- J6 pad 4: Net-(J6-Pad4) -> (no net)
- MX18 pad 1: Net-(J4-Pad4) -> Net-(J3-Pad1)
- MX18 pad 2: Net-(J4-Pad3) -> Net-(J3-Pad2)
- MX22 pad 1: Net-(J4-Pad1) -> Net-(J3-Pad4)
- MX22 pad 2: Net-(J4-Pad2) -> Net-(J3-Pad3)
- MX26 pad 1: Net-(J6-Pad4) -> Net-(J5-Pad1)
- MX26 pad 2: Net-(J6-Pad3) -> Net-(J5-Pad2)
- MX30 pad 1: Net-(J6-Pad1) -> Net-(J5-Pad4)
- MX30 pad 2: Net-(J6-Pad2) -> Net-(J5-Pad3)
Routing:
- net Net-(J8-Pad1): track 0.00 -> 144.9 mm
- net Net-(J1-Pad1): track 0.00 -> 139.9 mm
- net Net-(J8-Pad3): track 0.00 -> 132.7 mm
- net Net-(J8-Pad2): track 0.00 -> 127.9 mm
- net Net-(J1-Pad3): track 0.00 -> 126.8 mm
- net Net-(J1-Pad2): track 0.00 -> 120.8 mm
- net Net-(J1-Pad8): track 0.00 -> 100.4 mm
- net Net-(J8-Pad4): track 0.00 -> 100.2 mm
- net Net-(J8-Pad8): track 0.00 -> 98.3 mm
- net Net-(J1-Pad16): track 0.00 -> 95.4 mm
- net Net-(J1-Pad12): track 0.00 -> 94.6 mm
- net Net-(J8-Pad12): track 0.00 -> 94.2 mm
- net Net-(J8-Pad16): track 0.00 -> 93.9 mm
- net Net-(J1-Pad4): track 0.00 -> 92.1 mm
- net Net-(J1-Pad7): track 0.00 -> 78.4 mm
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Other:
- outline, holes or cut-outs redrawn

Commit message: Left side roughed in
Parts:
- C1, C10, C2, C3, C4, C5, C6, C7, C8, C9, D1, D10, D11, D12, D13, D14, D15, D16, D17, D18, D19, D2, D20, D21, D22, D23, D24, D25, D26, D27, D28, D29, D3, D30, D31, D32, D33, D34, D35, D36, D37, D38, D39, D4, D40, D41, D42, D43, D44, D5, D6, D7, D8, D9, F1, R1, R2, R3, R4, SW1, U1, USB1, Y1: moved to B.Cu
- moved D24 211.6 mm to (196.8, -136.1)
- moved D28 211.6 mm to (191.0, -136.1)
- moved D36 211.6 mm to (168.0, -136.1)
- moved D37 211.6 mm to (173.8, -136.1)
- moved D43 211.6 mm to (162.3, -136.1)
- moved D44 211.6 mm to (179.5, -136.1)
- moved D27 210.7 mm to (191.0, -139.4)
- moved D31 210.7 mm to (173.8, -139.4)
- moved D33 210.7 mm to (179.5, -139.4)
- moved D35 210.7 mm to (162.3, -139.4)
- moved D38 210.7 mm to (168.0, -139.4)
- moved D26 210.1 mm to (185.3, -142.8)
- moved D32 210.1 mm to (179.5, -142.8)
- moved D34 210.1 mm to (173.8, -142.8)
- moved D39 210.1 mm to (162.3, -142.8)
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Connections:
- J4 pad 1: (no net) -> COL7
- J4 pad 2: (no net) -> Net-(D18-Pad2)
- J4 pad 3: (no net) -> Net-(D19-Pad2)
- J4 pad 4: (no net) -> COL6
- J6 pad 1: (no net) -> COL5
- J6 pad 2: (no net) -> Net-(D29-Pad2)
- J6 pad 3: (no net) -> Net-(D30-Pad2)
- J6 pad 4: (no net) -> COL4
Routing:
- net GND: track 0.00 -> 151.2 mm, vias 0 -> 2
- net COL7: track 0.00 -> 149.0 mm, vias 0 -> 2
- net COL6: track 0.00 -> 147.4 mm, vias 0 -> 1
- net COLB: track 0.00 -> 118.5 mm, vias 0 -> 1
- net COLA: track 0.00 -> 115.5 mm, vias 0 -> 1
- net COL8: track 0.00 -> 113.4 mm, vias 0 -> 2
- net COL9: track 0.00 -> 113.1 mm, vias 0 -> 2
- net +5V: track 0.00 -> 79.5 mm, vias 0 -> 3
- net VCC: track 0.00 -> 71.9 mm, vias 0 -> 6
- net Net-(J3-Pad4): track 2.89 -> 66.8 mm
- net COL5: track 0.00 -> 58.7 mm
- net Net-(J5-Pad2): track 4.38 -> 61.2 mm
- net COL4: track 0.00 -> 54.7 mm
- net Net-(D5-Pad2): track 0.00 -> 53.3 mm
- net Net-(D16-Pad2): track 0.00 -> 52.5 mm
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Other:
- net class Power added: clearance 0.2, trace_width 0.6, via_dia 0.8, via_drill 0.4

Commit message: Laid out, ready for the pre-order inspection
Parts:
- moved D24 112.7 mm to (84.5, -126.7), turned to 90 degrees
- moved D27 100.2 mm to (91.7, -126.7), turned to 90 degrees
- moved D26 98.7 mm to (86.9, -135.3), turned to 90 degrees
- moved D23 90.0 mm to (84.5, -135.3), turned to 90 degrees
- moved D32 88.2 mm to (91.7, -135.3), turned to 90 degrees
- moved D25 87.0 mm to (105.4, -111.8), turned to 90 degrees
- moved D33 85.5 mm to (94.1, -135.3), turned to 90 degrees
- moved D31 84.6 mm to (89.3, -135.3), turned to 90 degrees
- moved D28 81.7 mm to (113.0, -111.8), turned to 90 degrees
- moved D37 80.2 mm to (94.1, -126.7), turned to 90 degrees
- moved D36 79.3 mm to (89.3, -126.7), turned to 90 degrees
- moved D34 77.6 mm to (96.5, -135.3), turned to 90 degrees
- moved D35 76.5 mm to (86.9, -126.7), turned to 90 degrees
- moved D40 74.5 mm to (100.3, -111.8), turned to 90 degrees
- moved D38 72.6 mm to (96.5, -126.7), turned to 90 degrees
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Routing:
- net COL4: track 54.7 -> 244.6 mm
- net ROW3: track 0.00 -> 138.9 mm, vias 0 -> 2
- net COL5: track 58.7 -> 179.6 mm, vias 0 -> 2
- net ROW2: track 0.00 -> 117.8 mm, vias 0 -> 3
- net COL2: track 0.00 -> 116.1 mm, vias 0 -> 2
- net COL3: track 0.00 -> 104.4 mm, vias 0 -> 4
- net COL1: track 0.00 -> 103.8 mm, vias 0 -> 2
- net COL0: track 0.00 -> 102.6 mm, vias 0 -> 2
- net ROW0: track 0.00 -> 83.6 mm, vias 0 -> 3
- net ROW1: track 0.00 -> 66.3 mm, vias 0 -> 2
- net Net-(D35-Pad2): track 0.00 -> 58.7 mm
- net Net-(D36-Pad2): track 0.00 -> 58.4 mm
- net Net-(D39-Pad2): track 0.00 -> 53.7 mm
- net Net-(D41-Pad2): track 0.00 -> 51.8 mm
- net Net-(D40-Pad2): track 0.00 -> 51.5 mm
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- added copper zone on B.Cu, net GND
Other:
- board text added: "Thumbs Up! Саша Карманов Alexander (Sasha) Karmanov January 2022 u/ak66666 https://github.com/ak66666/ThumbsUpUnsplit"
